File: electrical/Schematics.kicad_pcb (KiCad board)
At the start: 2 copper layers, 77.5 x 65 mm, 20 parts, among them J1 12V_IN, J2 RGB_STRIP_1, J3 WHITE_STRIP_1, J4 WHITE_STRIP_2, J5 RGB_STRIP_2, Q1 IRLB8721PBF, Q3 IRLB8721PBF, SW2 BTN, U1 L7805, U2 NodeMCU-ESP32-30pin

Commit message: update schematic to match actual GPIO assignments
Move signal connections from IO16/IO17/IO18/IO19 (right side) to
IO26/IO13/IO27/IO25 (left side) matching the working build.
PCB pad nets updated accordingly — traces need re-routing.

Co-Authored-By: Claude Opus 4.6 (1M context) <noreply@anthropic.com>
Connections:
- U2 pad 10: unconnected-(U2-IO26-Pad10) -> /RGB_DATA_1
- U2 pad 11: unconnected-(U2-IO27-Pad11) -> /WHITE_PWM_1
- U2 pad 14: unconnected-(U2-IO13-Pad14) -> /RGB_DATA_2
- U2 pad 23: /WHITE_PWM_2 -> unconnected-(U2-IO19-Pad23)
- U2 pad 24: /WHITE_PWM_1 -> unconnected-(U2-IO18-Pad24)
- U2 pad 26: /RGB_DATA_2 -> unconnected-(U2-IO17-Pad26)
- U2 pad 27: /RGB_DATA_1 -> unconnected-(U2-IO16-Pad27)
- U2 pad 9: unconnected-(U2-IO25-Pad9) -> /WHITE_PWM_2
Changed lines of the file:
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@@
 			(layers "*.Cu" "*.Mask")
 			(remove_unused_layers no)
-			(net "unconnected-(U2-IO25-Pad9)")
+			(net "/WHITE_PWM_2")
 			(pinfunction "IO25_9")
-			(pintype "bidirectional+no_connect")
+			(pintype "bidirectional")
 		)
 		(pad "10" thru_hole oval
@@
 			(layers "*.Cu" "*.Mask")
 			(remove_unused_layers no)
-			(net "unconnected-(U2-IO26-Pad10)")
+			(net "/RGB_DATA_1")
 			(pinfunction "IO26_10")
-			(pintype "bidirectional+no_connect")
+			(pintype "bidirectional")
 		)
 		(pad "11" thru_hole oval
@@
 			(layers "*.Cu" "*.Mask")
 			(remove_unused_layers no)
-			(net "unconnected-(U2-IO27-Pad11)")
+			(net "/WHITE_PWM_1")
 			(pinfunction "IO27_11")
-			(pintype "bidirectional+no_connect")
+			(pintype "bidirectional")
 		)
 		(pad "12" thru_hole oval
@@
 			(layers "*.Cu" "*.Mask")
 			(remove_unused_layers no)
-			(net "unconnected-(U2-IO13-Pad14)")
+			(net "/RGB_DATA_2")
 			(pinfunction "IO13_14")
-			(pintype "bidirectional+no_connect")
+			(pintype "bidirectional")
 		)
 		(pad "15" thru_hole oval
@@
 			(layers "*.Cu" "*.Mask")
 			(remove_unused_layers no)
-			(net "/WHITE_PWM_2")
+			(net "unconnected-(U2-IO19-Pad23)")
 			(pinfunction "IO19_23")
-			(pintype "bidirectional")
+			(pintype "bidirectional+no_connect")
 		)
 		(pad "24" thru_hole oval
@@
 			(layers "*.Cu" "*.Mask")
 			(remove_unused_layers no)
-			(net "/WHITE_PWM_1")
+			(net "unconnected-(U2-IO18-Pad24)")
 			(pinfunction "IO18_24")
-			(pintype "bidirectional")
+			(pintype "bidirectional+no_connect")
 		)
 		(pad "25" thru_hole oval
@@
 			(layers "*.Cu" "*.Mask")
 			(remove_unused_layers no)
-			(net "/RGB_DATA_2")
+			(net "unconnected-(U2-IO17-Pad26)")
 			(pinfunction "IO17_26")
-			(pintype "bidirectional")
+			(pintype "bidirectional+no_connect")
 		)
 		(pad "27" thru_hole oval
@@
 			(layers "*.Cu" "*.Mask")
 			(remove_unused_layers no)
-			(net "/RGB_DATA_1")
+			(net "unconnected-(U2-IO16-Pad27)")
 			(pinfunction "IO16_27")
-			(pintype "bidirectional")
+			(pintype "bidirectional+no_connect")
 		)
 		(pad "28" thru_hole oval
