File: electrical/Schematics.kicad_sch (KiCad schematic)
At the start: 20 parts, among them J1 12V_IN, J2 RGB_STRIP_1, J3 WHITE_STRIP_1, J4 WHITE_STRIP_2, J5 RGB_STRIP_2, Q1 IRLB8721PBF, Q3 IRLB8721PBF, SW2 BTN, U1 L7805, U2 NodeMCU-ESP32-30pin

Commit message: update schematic to match actual GPIO assignments
Move signal connections from IO16/IO17/IO18/IO19 (right side) to
IO26/IO13/IO27/IO25 (left side) matching the working build.
PCB pad nets updated accordingly — traces need re-routing.

Co-Authored-By: Claude Opus 4.6 (1M context) <noreply@anthropic.com>
Connections:
- net RGB_DATA_1: now also U2.10 (IO26); no longer U2.27 (IO16)
- net RGB_DATA_2: now also U2.14 (IO13); no longer U2.26 (IO17)
- net WHITE_PWM_1: now also U2.11 (IO27); no longer U2.24 (IO18)
- net WHITE_PWM_2: now also U2.9 (IO25); no longer U2.23 (IO19)
Changed lines of the file:
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@@
 	)
 	(no_connect
-		(at 124.46 63.5)
-	)
-	(no_connect
-		(at 124.46 73.66)
+		(at 160.02 66.04)
+	)
+	(no_connect
+		(at 160.02 68.58)
 	)
 	(no_connect
@@
 	)
 	(no_connect
-		(at 124.46 60.96)
+		(at 160.02 60.96)
 	)
 	(no_connect
@@
 	)
 	(no_connect
-		(at 124.46 66.04)
+		(at 160.02 58.42)
 	)
 	(no_connect
@@
 	(wire
 		(pts
-			(xy 160.02 68.58) (xy 165.1 68.58)
+			(xy 124.46 63.5) (xy 116.84 63.5)
 		)
 		(stroke
@@
 	(wire
 		(pts
-			(xy 160.02 66.04) (xy 165.1 66.04)
+			(xy 124.46 73.66) (xy 116.84 73.66)
 		)
 		(stroke
@@
 	(wire
 		(pts
-			(xy 160.02 60.96) (xy 165.1 60.96)
+			(xy 124.46 66.04) (xy 116.84 66.04)
 		)
 		(stroke
@@
 	(wire
 		(pts
-			(xy 160.02 58.42) (xy 165.1 58.42)
+			(xy 124.46 60.96) (xy 116.84 60.96)
 		)
 		(stroke
@@
 	)
 	(label "RGB_DATA_2"
-		(at 165.1 66.04 0)
+		(at 116.84 73.66 180)
 		(effects
 			(font
 				(size 1.27 1.27)
 			)
-			(justify left bottom)
+			(justify right bottom)
 		)
 	)
@@
 	)
 	(label "WHITE_PWM_1"
-		(at 165.1 60.96 0)
+		(at 116.84 66.04 180)
 		(effects
 			(font
 				(size 1.27 1.27)
 			)
-			(justify left bottom)
+			(justify right bottom)
 		)
 	)
 	(label "WHITE_PWM_2"
-		(at 165.1 58.42 0)
+		(at 116.84 60.96 180)
 		(effects
 			(font
 				(size 1.27 1.27)
 			)
-			(justify left bottom)
+			(justify right bottom)
 		)
 	)
 	(label "RGB_DATA_1"
-		(at 165.1 68.58 0)
+		(at 116.84 63.5 180)
 		(effects
 			(font
 				(size 1.27 1.27)
 			)
-			(justify left bottom)
-		)
-	)
+			(justify right bottom)
+		)
+	)
